File: Eagle_Workshop_Files/Workshop_Projects/Works_009.sch (EAGLE design)
At the start: 0 parts

Commit message: Added Works_009 and Works_009_a.sch
Parts:
- added U1: 328P, SparkFun-IC-Microcontroller:ATMEGA328P_PDIP
Other:
- note added: "AtMega328P 32KB of Programmable Flash Memory 1KB of EEPROM 2KB of SRAM 10bit ADC Most single clock cycle execution Up to 20MIPS Throughput at 20MHz"
- note added: "These are the analog input pins. Notice the pin 27 and 28, these are the I2C pins. Which means if these pins are not used as analog input pins, it works as I2C pins."
- note added: "These are the digital input/output pins. Notice the names in parentheses; those are the secondary usage pin. For example, pin 17~19 are used to program the microcontrller when not used. Otherwise, these pins can be used as regular digitial input/output pins."
- note added: "These are the power related pins. Connect appropriate power to these pins to supply power to your microcontroller."
- note added: "This is the external clock input pin. Remember, all CPUs need clock to properly operate. Faster the clock, faster the instructions are executed. Although AtMega chips have built-in internal clocks, they are slow(8Mhz) and inaccurate; which means it is always good idea to have external clock so the microcontroller can execute instructions without any delay."
- note added: "This is the hardware reset pin. Notice the small circle on the pin; this indicates this pin is active-low pin. Active-low pins are activated by pulling the pin to ground(GND)."
- note added: "Works_009 We will start talking about AtMega328P and how to wire it to make it work."
