File: Eagle_Workshop_Files/Workshop_Projects/Example_A.sch (EAGLE design)
At the start: 34 parts, among them J1 +9VDC, M1 MOTOR10MM, Q1 MOSFET_PCH-SI2309DS, Q2 MOSFET_PCH-SI2309DS, Q3 MOSFET_PCH-SI2309DS, Q4 MOSFET-NCH-PSMN7R0, Q5 MOSFET-NCH-PSMN7R0, Q6 MOSFET-NCH-FQP30N06L, Q7 MOSFET-NCH-FQP30N06L, U1 5V, U2 3V3

Commit message: Updated Example_A
Parts:
- added BT1: (no value), SparkFun-Retired:BATTERYFOB
- added C6: (no value), rcl:C-USC0805
- added J3: (no value), SparkFun-Connectors:CONN_023.5MM_LOCK
- added K1: RELAY-SPDT-JZC-11F, SparkFun-Electromechanical:RELAY-SPDT-JZC-11F
- added LS1: BUZZER-PTH, SparkFun-Electromechanical:BUZZER-PTH
- added R10, R11: 100k, SparkFun-Resistors:RESISTOR0805
- added R12: 1M, rcl:R-EU_R0805
- added S4, S5: MOMENTARY-SWITCH-SPST-SMD-RIGHT-ANGLE, SparkFun-Switches:MOMENTARY-SWITCH-SPST-SMD-RIGHT-ANGLE
- added U$1: ATTINY84ATTINY84-20PU, SparkFun-IC-Microcontroller:ATTINY84ATTINY84-20PU
- added Y1: (no value), SparkFun-Clocks:RESONATORSMD-7.4X3.4
Connections:
- new net N$10: U$1.(PCINT6/OC1A/SDA/MOSI/ADC6)PA6
- new net N$11: U$1.(PCINT4/T1/SCL/USCK/ADC4)PA4
- new net N$7: K1.NO, LS1.2
- new net N$9: K1.MAIN, S4.1
- new net RESET: R11.2, S5.1, U$1.(PCINT11/~RESET/DW)PB3
- new net XTAL1: R12.1, U$1.(PCINT8/XTAL1/CLKI)PB0, Y1.1
- new net XTAL2: R12.2, U$1.(PCINT9/XTAL2)PB1, Y1.3
- net 3.3V: now also S4.2
- net 5V: now also C2.1, C6.1, R11.1, U$1.VCC, U1.OUT, U1.OUT@1
- net GND: now also BT1.-, C6.2, J3.2, K1.COIL2, LS1.1, R10.1, S5.2, U$1.GND, Y1.2
- net N$5: now also K1.NC, R10.2; no longer C2.1, U1.OUT, U1.OUT@1
- net REC: now also U$1.(PCINT10/INT0/OC0A/CKOUT)PB2
- net VOUT: now also K1.COIL1
- net V_BATT: now also BT1.+, J3.1
Other:
- note added: "1: 2: 3: 4: 5: 6: 7: 8: 9: 10:"
- note added: "Battery"
- note added: "Controller"
- note added: "External Clock"
- note added: "Fig. 1"
- note added: "Fig. 10"
- note added: "Fig. 11"
- note added: "Fig. 12"
- note added: "Fig. 2"
- note added: "Fig. 3"
- note added: "Fig. 4"
- note added: "Fig. 5"
- note added: "Fig. 6"
- note added: "Fig. 7"
- note added: "Fig. 8"
- note added: "Fig. 9"
- note added: "Fuse Tester"
- note added: "Global Note (Unless Otherwise Specified) Resistor: 10k (Except r2) LED: Red Capacitor: 0.1uF"
- note added: "List Common Rules for Schematic Design (There are 10)"
- note added: "List any error(s) in Example_A Schematic. If there is no erro(s), put "No Error". Also, if figure is using a certain common sub-circuit, list them as well."
- note added: "Reset"
- note added: "Single Cell Li-Ion/Poly Only"
