File: Eagle_Workshop_Files/Workshop_Projects/Example_B.sch (EAGLE design)
At the start: 43 parts, among them IC1 ATTINY10, J2 AVR SPI PROG 3X2PTH, M1 MOTOR10MM, Q1 MOSFET_PCH-SI2309DS, Q2 MOSFET_PCH-SI2309DS, Q3 MOSFET-NCH-FDD8780, Q4 MOSFET-NCH-FDD8780, U1 TINY85-20-DIP, Y1 8MHz

Commit message: Added Example B
Parts:
- D1: value 4.1V -> ?V
- U1: value TINY85-20-DIP -> ATTINY85
Other:
- note added: "-Which Circuit Design Rule Can We Apply?"
- note added: "Extra Points -On the Schematic, Label Anything That is Missing. (Resistance, Capacitance, Missing Net Label, etc.) Write them on the Schematic Sheet."
- note added: "Fig. 10 -What Type of Diodie is Used?"
- note added: "Fig. 11 and 12 -(True or False) Figure 11 and 12 has full connection for all isolated nets"
- note added: "Fig. 13 -List Diode and Their Type(s) -What Type of Fuse is F1? -If We Want Short-Cirtcuit Protection for 12V Output, Which Component Should We Use? -Where Would We Place that Component at?"
- note added: "Fig. 14 -What Common Sub-Circuit is Used in The Figure? -For Q1~Q4, Define Type of Transistor and Their Type (That is, if BJT, is it NPN/PNP, or if it is FET, is it P-Channel/N-Channel?)"
- note added: "Fig. 2 -What is the type of the diode(D1)? -If we want VREF of 3.3V, what should be our Zener Voltage should be(Ignore voltage drop through R5)?"
- note added: "Fig. 3 -Which Circuit Design Rule Does the Figure Violate?"
- note added: "Fig. 4 -Which Circuit Design Rule Does the Figure Violate?"
- note added: "Fig. 5 -Which Circuit Design Rule Does the Figure Violate? -List Any Common Sub-Circuit"
- note added: "Fig. 6 - Which Circuit Design Rule Does the Figure Violate? -What type of diode is D5? -What type of switch is S1?"
- note added: "Fig. 7 -Which Circuit Design Rule Does the Figure Violate?"
- note added: "Fig. 8 -What is Missing in The Figure?"
- note added: "Fig. 9 -What Common Sub-Circuit is Used in The Figure?"
Changed lines of the file:
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@@
 <parts>
 <part name="FRAME1" library="frames" library_urn="urn:adsk.eagle:library:229" deviceset="LETTER_L" device=""/>
-<part name="D1" library="SparkFun-DiscreteSemi" deviceset="DIODE-ZENER" device="-MMSZ5232BS" value="4.1V"/>
+<part name="D1" library="SparkFun-DiscreteSemi" deviceset="DIODE-ZENER" device="-MMSZ5232BS" value="?V"/>
 <part name="D2" library="SparkFun-DiscreteSemi" deviceset="DIODE-SCHOTTKY" device="-SS14" value=""/>
 <part name="D4" library="SparkFun-LED" deviceset="LED-WHITE" device="1206" value="WHITE"/>
@@
 <part name="GND1" library="SparkFun-PowerSymbols" deviceset="GND" device=""/>
 <part name="SUPPLY2" library="SparkFun-PowerSymbols" deviceset="VCC" device=""/>
-<part name="U1" library="SparkFun-Retired" deviceset="ATTINY45" device="TINY85-20-DIP" value="TINY85-20-DIP"/>
+<part name="U1" library="SparkFun-Retired" deviceset="ATTINY45" device="TINY85-20-DIP" value="ATTINY85"/>
 <part name="Y1" library="SparkFun-Clocks" deviceset="RESONATOR-8MHZ" device="SMD_3.2X1.3" value="8MHz"/>
 <part name="GND2" library="SparkFun-PowerSymbols" deviceset="GND" device=""/>
@@
 <part name="GND16" library="SparkFun-PowerSymbols" deviceset="GND" device=""/>
 <part name="GND17" library="SparkFun-PowerSymbols" deviceset="GND" device=""/>
+<part name="FRAME2" library="frames" library_urn="urn:adsk.eagle:library:229" deviceset="LETTER_P" device=""/>
 </parts>
 <sheets>
@@
 <instance part="Y1" gate="G$1" x="73.66" y="175.26" rot="R270"/>
 <instance part="GND2" gate="1" x="60.96" y="175.26" rot="R270"/>
-<instance part="J2" gate="G$1" x="106.68" y="172.72"/>
-<instance part="GND3" gate="1" x="127" y="170.18" rot="R90"/>
-<instance part="SUPPLY3" gate="G$1" x="124.46" y="175.26" rot="R270"/>
+<instance part="J2" gate="G$1" x="114.3" y="172.72" smashed="yes" rot="MR0">
+<attribute name="NAME" x="119.38" y="178.308" size="1.778" layer="95" font="vector" rot="MR0"/>
+<attribute name="VALUE" x="129.54" y="165.354" size="1.778" layer="96" font="vector" rot="MR0"/>
+</instance>
+<instance part="GND3" gate="1" x="93.98" y="170.18" rot="MR90"/>
+<instance part="SUPPLY3" gate="G$1" x="96.52" y="175.26" rot="MR270"/>
 <instance part="C1" gate="G$1" x="139.7" y="170.18" rot="MR0"/>
 <instance part="GND4" gate="1" x="139.7" y="157.48"/>
@@
 <instance part="D11" gate="G$1" x="45.72" y="86.36" rot="R90"/>
 <instance part="R4" gate="G$1" x="40.64" y="91.44"/>
-<instance part="R5" gate="G$1" x="33.02" y="175.26"/>
+<instance part="R5" gate="G$1" x="33.02" y="175.26" smashed="yes">
+<attribute name="NAME" x="31.75" y="176.7586" size="1.778" layer="95"/>
+<attribute name="VALUE" x="29.21" y="171.958" size="1.778" layer="96"/>
+</instance>
 <instance part="GND14" gate="1" x="50.8" y="170.18" rot="R90"/>
 <instance part="SUPPLY9" gate="G$1" x="50.8" y="93.98"/>
@@
 <segment>
 <pinref part="J2" gate="G$1" pin="2"/>
-<wire x1="116.84" y1="175.26" x2="124.46" y2="175.26" width="0.1524" layer="91"/>
+<wire x1="104.14" y1="175.26" x2="96.52" y2="175.26" width="0.1524" layer="91"/>
 <pinref part="SUPPLY3" gate="G$1" pin="VCC"/>
 </segment>
@@
 <segment>
 <pinref part="J2" gate="G$1" pin="6"/>
-<wire x1="116.84" y1="170.18" x2="124.46" y2="170.18" width="0.1524" layer="91"/>
+<wire x1="104.14" y1="170.18" x2="96.52" y2="170.18" width="0.1524" layer="91"/>
 <pinref part="GND3" gate="1" pin="GND"/>
 </segment>
@@
 <segment>
 <pinref part="J2" gate="G$1" pin="5"/>
-<wire x1="99.06" y1="170.18" x2="91.44" y2="170.18" width="0.1524" layer="91"/>
-<label x="91.44" y="170.18" size="1.778" layer="95"/>
+<wire x1="121.92" y1="170.18" x2="129.54" y2="170.18" width="0.1524" layer="91"/>
+<label x="129.54" y="170.18" size="1.778" layer="95" rot="MR0"/>
 </segment>
 <segment>
@@
 <segment>
 <pinref part="J2" gate="G$1" pin="1"/>
-<wire x1="99.06" y1="175.26" x2="91.44" y2="175.26" width="0.1524" layer="91"/>
-<label x="91.44" y="175.26" size="1.778" layer="95"/>
+<wire x1="121.92" y1="175.26" x2="129.54" y2="175.26" width="0.1524" layer="91"/>
+<label x="129.54" y="175.26" size="1.778" layer="95" rot="MR0"/>
 </segment>
 <segment>
@@
 <segment>
 <pinref part="J2" gate="G$1" pin="3"/>
-<wire x1="99.06" y1="172.72" x2="91.44" y2="172.72" width="0.1524" layer="91"/>
-<label x="91.44" y="172.72" size="1.778" layer="95"/>
+<wire x1="121.92" y1="172.72" x2="129.54" y2="172.72" width="0.1524" layer="91"/>
+<label x="129.54" y="172.72" size="1.778" layer="95" rot="MR0"/>
 </segment>
 <segment>
@@
 <segment>
 <pinref part="J2" gate="G$1" pin="4"/>
-<wire x1="116.84" y1="172.72" x2="124.46" y2="172.72" width="0.1524" layer="91"/>
-<label x="119.38" y="172.72" size="1.778" layer="95"/>
+<wire x1="104.14" y1="172.72" x2="96.52" y2="172.72" width="0.1524" layer="91"/>
+<label x="101.6" y="172.72" size="1.778" layer="95" rot="MR0"/>
 </segment>
 <segment>
@@
 </nets>
 </sheet>
+<sheet>
+<plain>
+<text x="2.54" y="246.38" size="1.778" layer="91">Fig. 1</text>
+<text x="2.54" y="243.84" size="1.778" layer="91">-Which Circuit Design Rule Can We Apply?</text>
+<text x="2.54" y="226.06" size="1.778" layer="91">Fig. 2
+-What is the type of the diode(D1)?
+-If we want VREF of 3.3V, what should be our Zener Voltage should be(Ignore voltage drop through R5)?</text>
+<text x="2.54" y="215.9" size="1.778" layer="91">Fig. 3
+-Which Circuit Design Rule Does the Figure Violate?</text>
+<text x="2.54" y="205.74" size="1.778" layer="91">Fig. 4
+-Which Circuit Design Rule Does the Figure Violate?</text>
+<text x="2.54" y="187.96" size="1.778" layer="91">Fig. 5
+-Which Circuit Design Rule Does the Figure Violate?
+-List Any Common Sub-Circuit</text>
+<text x="2.54" y="160.02" size="1.778" layer="91">Fig. 6
+- Which Circuit Design Rule Does the Figure Violate?
+-What type of diode is D5?
+-What type of switch is S1?</text>
+<text x="2.54" y="149.86" size="1.778" layer="91">Fig. 7
+-Which Circuit Design Rule Does the Figure Violate?</text>
+<text x="2.54" y="137.16" size="1.778" layer="91">Fig. 8
+-What is Missing in The Figure?</text>
+<text x="2.54" y="124.46" size="1.778" layer="91">Fig. 9
+-What Common Sub-Circuit is Used in The Figure?</text>
+<text x="2.54" y="111.76" size="1.778" layer="91">Fig. 10
+-What Type of Diodie is Used?</text>
+<text x="2.54" y="99.06" size="1.778" layer="91">Fig. 11 and 12
+-(True or False) Figure 11 and 12 has full connection for all isolated nets</text>
+<text x="2.54" y="63.5" size="1.778" layer="91">Fig. 13
+-List Diode and Their Type(s)
+-What Type of Fuse is F1?
+-If We Want Short-Cirtcuit Protection for 12V Output, Which Component Should We Use?
+-Where Would We Place that Component at?</text>
+<text x="2.54" y="43.18" size="1.778" layer="91">Fig. 14
+-What Common Sub-Circuit is Used in The Figure?
+-For Q1~Q4, Define Type of Transistor and Their Type
+(That is, if BJT, is it NPN/PNP, or if it is FET, is it P-Channel/N-Channel?)</text>
+<text x="2.54" y="25.4" size="1.778" layer="91">Extra Points
+-On the Schematic, Label Anything That is Missing.
+(Resistance, Capacitance, Missing Net Label, etc.)
+Write them on the Schematic Sheet.</text>
+</plain>
+<instances>
+<instance part="FRAME2" gate="G$1" x="0" y="0"/>
+<instance part="FRAME2" gate="G$2" x="83.82" y="0"/>
+</instances>
+<busses>
+</busses>
+<nets>
+</nets>
+</sheet>
 </sheets>
 </schematic>
 </drawing>
 <compatibility>
+<note version="6.3" minversion="6.2.2" severity="warning">
+Since Version 6.2.2 text objects can contain more than one line,
+which will not be processed correctly with this version.
+</note>
 <note version="8.2" severity="warning">
 Since Version 8.2, Eagle supports online libraries. The ids
