File: Eagle_Workshop_Files/Workshop_Projects/Works_009_a.sch (EAGLE design)
At the start: 0 parts

Commit message: Added #9a
Parts:
- added C1: 0.1uF, resistor:C-USC0805
- added D1: DIODE-BAS16J, SparkFun-DiscreteSemi:DIODE-BAS16J
- added R1: 4.7k, resistor:R-US_R0805
- added R2: 330, resistor:R-US_R0805
- added S1: SPST, SparkFun-Switches:MOMENTARY-SWITCH-SPST-SMD-5.2MM
- added U1: 328P, SparkFun-IC-Microcontroller:ATMEGA328P_PDIP
- added Y1: 16MHz, SparkFun-Clocks:RESONATOR-16MHZSMD_3.2X1.3
Connections:
- new net GND: C1.2, S1.2, U1.GND@1, U1.GND@2, Y1.2
- new net N$6: U1.PB6(XTAL1/TOSC1), Y1.1
- new net N$7: U1.PB7(XTAL2/TOSC2), Y1.3
- new net N$9: R2.1, S1.1
- new net VCC: C1.1, D1.A, D1.C, R1.1, R1.2, R2.2, U1.AREF, U1.AVCC, U1.PC6(/RESET), U1.VCC
Other:
- note added: "D1: 250mA/100V"
